Commit message: lab 3 submission

File: src/my_robot_description/urdf/gazebo_plugins.xacro (robot description, xacro)
@@ -3,4 +3,15 @@
     <xacro:property name="FOV" value="60" />
     <!--TODO Adding differential drive - add the DiffDrive plugin here.-->
+    <gazebo>
+        <plugin
+            filename="gz-sim-diff-drive-system"
+            name="gz::sim::systems::DiffDrive">
+            <left_joint>base_left_wheel_joint</left_joint>
+            <right_joint>base_right_wheel_joint</right_joint>
+            <wheel_separation>${base_width}</wheel_separation>
+            <wheel_radius>${wheel_radius}</wheel_radius>
+            <topic>cmd_vel</topic>
+        </plugin>
+    </gazebo>
     <!-- End Adding differential drive -->
     <gazebo reference="caster_wheel_link">

File: src/my_robot_description/urdf/my_robot.urdf.xacro (robot description, xacro)
@@ -50,4 +50,46 @@
     </link>
     <!--TODO Adding wheels links - add "right_wheel_link" and "left_wheel_link" here-->
+    <link name="right_wheel_link">
+        <xacro:cylinder_inertia
+            m="1"
+            r="${wheel_radius}"
+            l="${wheel_length}"
+            o_xyz="0 0 0"
+            o_rpy="${base_height / 2} 0 0"/>
+        <collision>
+            <origin xyz="0 0 0" rpy="${pi / 2} 0 0" />
+            <geometry>
+                <cylinder radius="${wheel_radius}" length="${wheel_length}" />
+            </geometry>
+        </collision>
+        <visual>
+            <origin xyz="0 0 0" rpy="${pi / 2} 0 0" />
+            <geometry>
+                <cylinder radius="${wheel_radius}" length="${wheel_length}" />
+            </geometry>
+            <material name="gray" />
+        </visual>
+    </link>
+    <link name="left_wheel_link">
+        <xacro:cylinder_inertia
+            m="1"
+            r="${wheel_radius}"
+            l="${wheel_length}"
+            o_xyz="0 0 0"
+            o_rpy="${base_height / 2} 0 0"/>
+        <collision>
+            <origin xyz="0 0 0" rpy="${pi / 2} 0 0" />
+            <geometry>
+                <cylinder radius="${wheel_radius}" length="${wheel_length}" />
+            </geometry>
+        </collision>
+        <visual>
+            <origin xyz="0 0 0" rpy="${pi / 2} 0 0" />
+            <geometry>
+                <cylinder radius="${wheel_radius}" length="${wheel_length}" />
+            </geometry>
+            <material name="gray" />
+        </visual>
+    </link>
     <!-- End Adding wheels links -->
     <link name="caster_wheel_link">
@@ -74,4 +116,16 @@
     </joint>
     <!-- TODO Adding wheels joints - add a joint to the base_link for each wheel-->
+    <joint name="base_right_wheel_joint" type="continuous">
+        <parent link="base_link" />
+        <child link="right_wheel_link" />
+        <origin xyz="0 -0.085 0" rpy="0 0 0" />
+        <axis xyz="0 1 0" />
+    </joint>
+    <joint name="base_left_wheel_joint" type="continuous">
+        <parent link="base_link" />
+        <child link="left_wheel_link" />
+        <origin xyz="0 0.085 0" rpy="0 0 0" />
+        <axis xyz="0 1 0" />
+    </joint>
     <!-- End Adding wheels joints -->
     <joint name="base_caster_wheel_joint" type="fixed">
